Commit message: Dual-ukf system and general fixes.

File: src/earendil_bot/description/camera.xacro (robot description, xacro)
@@ -8,6 +8,6 @@
         <parent link="body_link"/>
         <child link="camera_link"/>
-        <!-- Placed at the front, sitting ON TOP of the rover body -->
-        <origin xyz="${body_link_x_dim/2} 0 0" rpy="0 0 0"/>
+        <!-- Placed at the front, sitting on top of the rover body -->
+        <origin xyz="${body_link_x_dim/2} 0 ${body_link_z_dim/2 + cam_height/2}" rpy="0 0 0"/>
     </joint>
     <link name="camera_link">
@@ -55,19 +55,28 @@
     <gazebo reference="camera_link">
         <material>Gazebo/Black</material>
-        <!-- RGB Camera Sensor (IMX219 specs scaled to 1080p for sim performance) -->
-        <sensor name="camera" type="camera">
+        <!-- RGB-D Camera Sensor -->
+        <!-- Publishes:
+             /camera/image_raw
+             /camera/camera_info
+             /camera/depth/image_raw
+             /camera/depth/camera_info
+             /camera/points
+        -->
+        <sensor name="camera" type="depth">
             <pose> 0 0 0 0 0 0 </pose>
             <visualize>true</visualize>
-            <update_rate>30</update_rate>
+            <update_rate>15</update_rate>
             <camera>
                 <horizontal_fov>1.274</horizontal_fov> <!-- 73 degrees horizontal FOV -->
                 <image>
                     <format>R8G8B8</format>
-                    <width>1920</width>
-                    <height>1080</height>
+                    <width>640</width>
+                    <height>480</height>
                 </image>
+                <depth_camera>
+                </depth_camera>
                 <clip>
                     <near>0.05</near>
-                    <far>32.0</far>
+                    <far>8.0</far>
                 </clip>
             </camera>
@@ -75,29 +84,6 @@
                 <camera_name>camera</camera_name>
                 <frame_name>camera_link_optical</frame_name>
-            </plugin>
-        </sensor>
-        <!-- IMU Sensor (ICM20948 specs) -->
-        <sensor name="imu_sensor" type="imu">
-            <always_on>true</always_on>
-            <update_rate>100</update_rate>
-            <visualize>true</visualize>
-            <imu>
-                <angular_velocity>
-                    <x><noise type="gaussian"><mean>0.0</mean><stddev>2e-4</stddev><bias_mean>0.0000075</bias_mean><bias_stddev>0.0000008</bias_stddev></noise></x>
-                    <y><noise type="gaussian"><mean>0.0</mean><stddev>2e-4</stddev><bias_mean>0.0000075</bias_mean><bias_stddev>0.0000008</bias_stddev></noise></y>
-                    <z><noise type="gaussian"><mean>0.0</mean><stddev>2e-4</stddev><bias_mean>0.0000075</bias_mean><bias_stddev>0.0000008</bias_stddev></noise></z>
-                </angular_velocity>
-                <linear_acceleration>
-                    <x><noise type="gaussian"><mean>0.0</mean><stddev>1.7e-2</stddev><bias_mean>0.1</bias_mean><bias_stddev>0.001</bias_stddev></noise></x>
-                    <y><noise type="gaussian"><mean>0.0</mean><stddev>1.7e-2</stddev><bias_mean>0.1</bias_mean><bias_stddev>0.001</bias_stddev></noise></y>
-                    <z><noise type="gaussian"><mean>0.0</mean><stddev>1.7e-2</stddev><bias_mean>0.1</bias_mean><bias_stddev>0.001</bias_stddev></noise></z>
-                </linear_acceleration>
-            </imu>
-            <plugin name="imu_plugin" filename="libgazebo_ros_imu_sensor.so">
-                <ros>
-                    <namespace>/imu</namespace>
-                    <remapping>~/out:=data</remapping>
-                </ros>
-                <initial_orientation_as_reference>false</initial_orientation_as_reference>
+                <min_depth>0.15</min_depth>
+                <max_depth>8.0</max_depth>
             </plugin>
         </sensor>

File: src/earendil_bot/description/lidar.xacro (robot description, xacro)
@@ -46,5 +46,5 @@
 			</scan>
 			<range>
-				<min>0.7</min>
+				<min>0.6</min>
 				<max>12.0</max>
 				<resolution>0.015</resolution>

File: src/earendil_bot/description/robot.urdf.xacro (robot description, xacro)
@@ -45,13 +45,4 @@
 <!-- Here we include the file that defines extra Gazebo options and motion control driver -->
 <xacro:include filename="$(find earendil_bot)/description/robot.gazebo" />
-<!-- ################################################################################ -->
-<!-- Dummy link -->
-<link name="dummy">
-</link>
-<joint name="dummy_joint" type="fixed">
-	<parent link="dummy"/>
-	<child link="base_footprint"/>
-	<origin rpy="0 0 0" xyz="0 0 0"/>
-</joint>
 <!-- START links and joints:  -->
 <!-- ################################################################################ -->
@@ -195,3 +186,6 @@
 <!-- Starting Camera / IMU -->
 <xacro:include filename="camera.xacro" />
+<!-- ################################################################################ -->
+<!-- Starting IMU -->
+<xacro:include filename="imu.xacro" />
 </robot>
